File: kicad/einkclock.kicad_pcb (KiCad board)
At the start: 2 copper layers, 61 parts, among them P1 SWD, Q1 IRLIB9343PBF, Q2 IRLIB9343PBF, Q3 IRLU120N, Q4 IRLU120N, U1 MCP1702-3302ETO, U2 MC33063A, U3 MC33063A, U4 MC78L15ACP, U5 MC79L15ACP, U6 ED060SC4V2, U7 LM358, U8 DCF77_Generic, U9 LPC1227FBD48/301, Y1 30M 12.5p, Y2 32.768k 12.5p

Commit message: Start PCB routing
Parts:
- removed R17: 100k, Resistors_THT:R_Axial_DIN0207_L6.3mm_D2.5mm_P10.16mm_Horizontal
- removed Y2: 32.768k 12.5p, Crystals:Crystal_Round_d3.0mm_Vertical
- added C23: 100n, Capacitors_THT:C_Disc_D4.3mm_W1.9mm_P5.00mm, F.Cu at (70.0, 31.4)
- added C24: 22p, Capacitors_THT:C_Disc_D4.3mm_W1.9mm_P5.00mm, F.Cu at (76.3, 39.0)
- added L3: 10µ, Resistors_THT:R_Axial_DIN0414_L11.9mm_D4.5mm_P20.32mm_Horizontal, F.Cu at (90.2, 102.9)
- added REF**: MountingHole_2.2mm_M2, Mounting_Holes:MountingHole_2.2mm_M2, F.Cu at (90.2, 110.5)
- added REF**: MountingHole_2.2mm_M2, Mounting_Holes:MountingHole_2.2mm_M2, F.Cu at (90.2, 17.8)
- added REF**: MountingHole_2.2mm_M2, Mounting_Holes:MountingHole_2.2mm_M2, F.Cu at (17.8, 110.5)
- added REF**: MountingHole_2.2mm_M2, Mounting_Holes:MountingHole_2.2mm_M2, F.Cu at (17.8, 17.8)
- C1, C10, C2, C9: footprint Capacitors_THT:CP_Radial_Tantal_D4.5mm_P2.50mm -> Capacitors_THT:CP_Radial_D8.0mm_P5.00mm
- C11, C12, C13, C14, C15, C21, C3, C4, C5, C6, C7, C8: footprint Capacitors_THT:CP_Radial_Tantal_D4.5mm_P2.50mm -> Capacitors_THT:C_Disc_D4.3mm_W1.9mm_P5.00mm
- C16: value 4.7u -> 100n; footprint Capacitors_THT:CP_Radial_Tantal_D4.5mm_P2.50mm -> Capacitors_THT:C_Disc_D4.3mm_W1.9mm_P5.00mm
- C17, C18, C22: value 22p -> 100n; footprint Capacitors_THT:CP_Radial_Tantal_D4.5mm_P2.50mm -> Capacitors_THT:C_Disc_D4.3mm_W1.9mm_P5.00mm
- C19: value 100n -> 100µ; footprint Capacitors_THT:CP_Radial_Tantal_D4.5mm_P2.50mm -> Capacitors_THT:CP_Radial_D8.0mm_P5.00mm
- C20: value 100n -> 4.7u; footprint Capacitors_THT:CP_Radial_Tantal_D4.5mm_P2.50mm -> Capacitors_THT:CP_Radial_D8.0mm_P5.00mm
- L1, L2: footprint Resistors_THT:R_Axial_DIN0411_L9.9mm_D3.6mm_P15.24mm_Horizontal -> Resistors_THT:R_Axial_DIN0516_L15.5mm_D5.0mm_P20.32mm_Horizontal
- Q1, Q2: footprint TO_SOT_Packages_THT:TO-220_Neutral123_Horizontal -> TO_SOT_Packages_THT:TO-220_Horizontal
- Q3, Q4: footprint TO_SOT_Packages_THT:TO-220_Neutral123_Horizontal -> TO_SOT_Packages_THT:TO-251_IPAK_Vertical
- R10: value 2k -> 200k
- R11: value 2k -> 10k
- R12: value 47k -> 2.2k
- R13: value 100k -> 2.2k
- R14: value 100k -> 47k
- R2, R4: footprint Resistors_THT:R_Axial_DIN0207_L6.3mm_D2.5mm_P10.16mm_Horizontal -> Resistors_THT:R_Axial_DIN0516_L15.5mm_D5.0mm_P20.32mm_Horizontal
- R8: value 200k -> 100k
- R9: value 10k -> 100k
- RV1: footprint Potentiometers:Potentiometer_Alps-RK16-single -> Potentiometers:Potentiometer_Alps_RK09K_Horizontal
- U1: footprint TO_SOT_Packages_THT:TO-220_Neutral123_PadsOnly -> TO_SOT_Packages_THT:TO-92_Inline_Narrow_Oval
- U2, U3, U7: footprint Housings_DIP:DIP-8_W7.62mm -> Housings_DIP:DIP-8_W7.62mm_LongPads
- U4, U5: footprint TO_SOT_Packages_THT:TO-92_Inline_Wide -> TO_SOT_Packages_THT:TO-92_Inline_Narrow_Oval
- U6: footprint Socket_Strips:Socket_Strip_Straight_1x38 -> kaini:Hirose_FH26-39S-0.3SHW
- U8: footprint Socket_Strips:Socket_Strip_Straight_1x04 -> kaini:Reichelt_DCF77_Module
- U9: footprint kaini:QFP48 Adapter -> Housings_QFP:LQFP-48_7x7mm_Pitch0.5mm
- Y1: value 30M 12.5p -> 32.768k 12.5p; footprint Crystals:Crystal_HC49-U_Vertical -> Crystals:Crystal_AT310_d3.0mm_l10.0mm_Vertical
- moved L2 142.0 mm to (31.8, 85.1)
- moved U6 141.8 mm to (89.1, 51.0), turned to 270 degrees
- moved C11 135.9 mm to (50.8, 35.1), turned to 90 degrees
- moved U9 122.3 mm to (73.7, 50.8)
- moved C2 119.9 mm to (26.7, 93.5), turned to 180 degrees
- moved R3 116.7 mm to (31.8, 80.0), turned to 90 degrees
- moved R1 114.9 mm to (31.8, 40.6), turned to 90 degrees
- moved L1 114.5 mm to (30.5, 64.8)
- moved C10 110.6 mm to (52.1, 96.0), turned to 90 degrees
- moved Q3 106.5 mm to (27.9, 43.2), turned to 270 degrees
- moved Q1 105.6 mm to (17.8, 48.4)
- moved R6 105.0 mm to (43.2, 40.6), turned to 90 degrees
- moved R8 103.1 mm to (27.9, 30.5), turned to 270 degrees
- moved U2 102.1 mm to (38.1, 59.7), turned to 180 degrees
- moved C4 100.8 mm to (17.8, 50.8), turned to 270 degrees
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Connections:
- C17 pad 1: GND -> +3V3
- C17 pad 2: Net-(C17-Pad2) -> GND
- C19 pad 1: GND -> Net-(C18-Pad1)
- C19 pad 2: +3V3 -> GND
- C20 pad 1: GND -> +3V3
- C20 pad 2: +3V3 -> GND
- C21 pad 1: GND -> Net-(C21-Pad1)
- C21 pad 2: Net-(C21-Pad2) -> GND
- C22 pad 1: Net-(C22-Pad1) -> GND
- C22 pad 2: GND -> +3V3
- P1 pad 6: Net-(P1-Pad6) -> (no net)
- P1 pad 8: Net-(P1-Pad8) -> (no net)
- Q1 pad 1: Net-(C1-Pad1) -> Net-(C4-Pad1)
- Q1 pad 2: Net-(C4-Pad1) -> Net-(C1-Pad1)
- Q2 pad 1: Net-(C2-Pad1) -> Net-(C5-Pad1)
- Q2 pad 2: Net-(C5-Pad1) -> Net-(C2-Pad1)
- Q3 pad 1: Net-(Q3-Pad1) -> /ONPOS
- Q3 pad 2: /ONPOS -> Net-(C4-Pad1)
- Q3 pad 3: Net-(C4-Pad1) -> Net-(Q3-Pad3)
- Q4 pad 1: Net-(Q4-Pad1) -> /ONNEG
- Q4 pad 2: /ONNEG -> Net-(C5-Pad1)
- Q4 pad 3: Net-(C5-Pad1) -> Net-(Q4-Pad3)
- R10 pad 1: GND -> /+22V
- R10 pad 2: Net-(Q3-Pad1) -> Net-(R10-Pad2)
- R11 pad 1: GND -> /-20V
- R11 pad 2: Net-(Q4-Pad1) -> Net-(R11-Pad2)
- R12 pad 1: Net-(R12-Pad1) -> GND
- R12 pad 2: /-15V -> Net-(Q3-Pad3)
- R13 pad 1: Net-(P1-Pad10) -> GND
- R13 pad 2: +3V3 -> Net-(Q4-Pad3)
- R14 pad 1: Net-(P1-Pad6) -> Net-(R14-Pad1)
- R14 pad 2: +3V3 -> /-15V
- R15 pad 1: Net-(P1-Pad2) -> Net-(R15-Pad1)
- R16 pad 1: Net-(R16-Pad1) -> Net-(P1-Pad10)
- R6 pad 1: Net-(R6-Pad1) -> Net-(R10-Pad2)
- R7 pad 1: Net-(R7-Pad1) -> Net-(R11-Pad2)
- R8 pad 1: /+22V -> GND
- R8 pad 2: Net-(R6-Pad1) -> /ONPOS
- R9 pad 1: /-20V -> GND
- R9 pad 2: Net-(R7-Pad1) -> /ONNEG
- RV1 pad 3: Net-(R12-Pad1) -> Net-(R14-Pad1)
- U2 pad 5: Net-(R6-Pad1) -> Net-(R10-Pad2)
- U3 pad 5: Net-(R7-Pad1) -> Net-(R11-Pad2)
- U5 pad 1: /-15V -> GND
- U5 pad 2: GND -> /-20V
- U5 pad 3: /-20V -> /-15V
- U8 pad 2: /TON -> GND
- U8 pad 4: +3V3 -> Net-(C18-Pad1)
- U9 pad 1: Net-(C17-Pad2) -> (no net)
- U9 pad 12: Net-(U9-Pad12) -> /TON
- U9 pad 13: Net-(U9-Pad13) -> (no net)
- U9 pad 14: Net-(U9-Pad14) -> /DON
- U9 pad 15: /DD0 -> /DD7
- U9 pad 16: /DD1 -> /DD6
- U9 pad 17: /DD2 -> /DD5
- U9 pad 18: /DD3 -> /DD4
- U9 pad 19: /DD4 -> /DD3
- U9 pad 2: Net-(C21-Pad2) -> (no net)
- U9 pad 20: /DD5 -> /DD2
- U9 pad 21: /DD6 -> /DD1
- U9 pad 22: /DD7 -> /DD0
- U9 pad 23: /DCL -> /DSPH
- U9 pad 24: /DLE -> /DOE
- U9 pad 25: /DOE -> /DLE
- U9 pad 26: /DSPH -> /TSIG
- U9 pad 27: /DON -> Net-(P1-Pad7)
- U9 pad 29: /DGMODE -> /DCL
- U9 pad 3: +3V3 -> (no net)
- U9 pad 32: /ONPOS -> /DGMODE
- U9 pad 33: /ONNEG -> /ONPOS
- U9 pad 34: Net-(U9-Pad34) -> (no net)
- U9 pad 35: Net-(U9-Pad35) -> (no net)
- U9 pad 36: Net-(U9-Pad36) -> (no net)
- U9 pad 37: Net-(U9-Pad37) -> (no net)
- U9 pad 38: Net-(U9-Pad38) -> (no net)
- U9 pad 39: Net-(R16-Pad1) -> Net-(R15-Pad1)
- U9 pad 4: /TSIG -> /ONNEG
- U9 pad 40: Net-(U9-Pad40) -> (no net)
- U9 pad 41: Net-(U9-Pad41) -> (no net)
- U9 pad 42: Net-(U9-Pad42) -> (no net)
- U9 pad 45: Net-(C22-Pad1) -> Net-(C24-Pad1)
- U9 pad 46: Net-(C18-Pad1) -> Net-(C21-Pad1)
- U9 pad 5: /TON -> (no net)
- U9 pad 6: Net-(U9-Pad6) -> (no net)
- U9 pad 7: Net-(U9-Pad7) -> (no net)
- U9 pad 8: Net-(U9-Pad8) -> (no net)
- U9 pad 9: Net-(U9-Pad9) -> (no net)
- Y1 pad 1: Net-(C17-Pad2) -> Net-(C21-Pad1)
- Y1 pad 2: Net-(C21-Pad2) -> Net-(C24-Pad1)
Routing:
- net GND: track 17.8 -> 234.7 mm, vias 0 -> 2
- net Net-(L1-Pad1): track 0.00 -> 57.9 mm
- net /-20V: track 0.00 -> 55.3 mm, vias 0 -> 1
- net +BATT: track 12.7 -> 67.6 mm
- net /+22V: track 0.00 -> 34.4 mm
- net Net-(C2-Pad1): track 0.00 -> 33.9 mm
- net Net-(C1-Pad1): track 0.00 -> 32.7 mm
- net Net-(D2-Pad1): track 0.00 -> 23.9 mm
- net Net-(R5-Pad1): track 0.00 -> 23.4 mm
- net Net-(R10-Pad2): track 0.00 -> 21.2 mm
- net Net-(C5-Pad1): track 0.00 -> 21.2 mm
- net Net-(C4-Pad1): track 0.00 -> 20.9 mm
- net Net-(R11-Pad2): track 0.00 -> 18.6 mm
- net Net-(R4-Pad1): track 0.00 -> 17.5 mm
- net /DON: track 0.00 -> 16.1 mm, vias 0 -> 3
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Other:
- board outline added: 80 x 100.3 mm
- net class Default: clearance 0.2 -> 0.15
- rule trace_clearance: 0.2 -> 0.15
- rule trace_min: 0.2 -> 0.15
- board text added: "+"
- board text added: "-"
