File: kicad/einkclock.sch (KiCad schematic (older format))
At the start: 61 parts, among them P1 SWD, Q1 IRLIB9343PBF, Q2 IRLIB9343PBF, Q3 IRLU120N, Q4 IRLU120N, U1 MCP1702-3302ETO, U2 MC33063A, U3 MC33063A, U4 MC78L15ACP, U5 MC79L15ACP, U6 ED060SC4V2, U7 LM358, U8 DCF77_Generic, U9 LPC1227FBD48/301, Y1 30M 12.5p, Y2 32.768k 12.5p

Commit message: Add fixes to KiCad schematc
Parts:
- removed C21: 22p, Capacitors_THT:CP_Radial_Tantal_D4.5mm_P2.50mm, symbol C
- removed Q1, Q2: IRLIB9343PBF, TO_SOT_Packages_THT:TO-220_Neutral123_Horizontal, symbol Q_PMOS_DGS
- removed Q3, Q4: IRLU120N, TO_SOT_Packages_THT:TO-220_Neutral123_Horizontal, symbol Q_NMOS_DGS
- removed R14, R15, R17: 100k, Resistors_THT:R_Axial_DIN0207_L6.3mm_D2.5mm_P10.16mm_Horizontal, symbol R
- removed U5: MC79L15ACP, TO_SOT_Packages_THT:TO-92_Inline_Wide, symbol MC78L15ACP
- removed Y1: 30M 12.5p, Crystals:Crystal_HC49-U_Vertical, symbol Crystal
- added C16: 100n, Capacitors_THT:CP_Radial_Tantal_D4.5mm_P2.50mm, symbol C
- added C18: 100n, symbol C
- added C19: 100µ, symbol CP
- added L3: 10µ, symbol L
- added Q1, Q2: IRLIB9343PBF, symbol Q_PMOS_GDS
- added Q3, Q4: IRLU120N, symbol Q_NMOS_GDS
- added R8, R9: 100k, symbol R
- added U5: MC79L15ACP, TO-220, symbol LM7905CT
- C17: value 22p -> 100n
- R12: renamed from R10; value 2k -> 2.2k
- R13: renamed from R11; value 2k -> 2.2k
- renumbered C16 to C20, C18 to C21, C19 to C22, C20 to C23, C22 to C24, R8 to R10, R9 to R11, R12 to R14, R16 to R15, R13 to R16, Y2 to Y1
Connections:
- net +3V3: now also C17.1, C16.1; no longer U8.4 (VCC), U9.3 (VREF_CMP)
- net +BATT: now also Q1.3 (S), Q2.3 (S)
- net -15V: now also U5.3 (OUT)
- net -20V: now also U5.2 (IN)
- net DON: now also U9.13 (PIO0_28*); no longer U9.27 (PIO0_12*)
- net DSPH: now also U9.32 (PIO0_17); no longer U9.26 (PIO0_11)
- net GND: now also C17.2, U8.2 (ON), C16.2, C18.2, C19.2, R8.1, R9.1, U5.1 (GND); no longer C17.1
- net ONNEG: now also U9.4 (PIO0_19), Q4.1 (G), R9.2; no longer U9.33 (PIO0_18)
- net ONPOS: now also U9.33 (PIO0_18), Q3.1 (G), R8.2; no longer U9.32 (PIO0_17)
- net TON: now also U9.14 (PIO0_29*), L3.2; no longer U8.2 (ON), U9.5 (PIO0_20)
- net TSIG: now also U9.26 (PIO0_11); no longer U9.4 (PIO0_19)
- net at R12.2: now also Q3.2 (D)
- net at C4.1, R1.1: now also Q1.1 (G), Q3.3 (S)
- net at C1.1, C4.2, R2.2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: now also Q1.2 (D)
- net at R13.2: now also Q4.2 (D)
- net at C5.1, R3.1: now also Q2.1 (G), Q4.3 (S)
- net at C2.1, C5.2, R4.2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: now also Q2.2 (D)
- net at U9.1 (XTALIN): no longer C17.2
- net at P1.7 (P7): now also U9.27 (PIO0_12*)
- new net: C18.1, C19.1, L3.1, U8.4 (VCC)
- no-connect marks 17 -> 19
Other:
- moved on the sheet: R16, U8

Commit message: Start PCB routing
Parts:
- C1, C10, C2, C20, C9: footprint Capacitors_THT:CP_Radial_Tantal_D4.5mm_P2.50mm -> Capacitors_THT:CP_Radial_D8.0mm_P5.00mm
- C11, C12, C13, C14, C15, C16, C17, C21, C22, C23, C24, C3, C4, C5, C6, C7, C8: footprint Capacitors_THT:CP_Radial_Tantal_D4.5mm_P2.50mm -> Capacitors_THT:C_Disc_D4.3mm_W1.9mm_P5.00mm
- C18: footprint (none) -> Capacitors_THT:C_Disc_D4.3mm_W1.9mm_P5.00mm
- C19: footprint (none) -> Capacitors_THT:CP_Radial_D8.0mm_P5.00mm
- L1, L2: footprint Resistors_THT:R_Axial_DIN0411_L9.9mm_D3.6mm_P15.24mm_Horizontal -> Resistors_THT:R_Axial_DIN0516_L15.5mm_D5.0mm_P20.32mm_Horizontal
- L3: footprint (none) -> Resistors_THT:R_Axial_DIN0414_L11.9mm_D4.5mm_P20.32mm_Horizontal
- Q1, Q2: footprint (none) -> TO_SOT_Packages_THT:TO-220_Horizontal
- Q3, Q4: footprint (none) -> TO_SOT_Packages_THT:TO-251_IPAK_Vertical
- R2, R4: footprint Resistors_THT:R_Axial_DIN0207_L6.3mm_D2.5mm_P10.16mm_Horizontal -> Resistors_THT:R_Axial_DIN0516_L15.5mm_D5.0mm_P20.32mm_Horizontal
- R8, R9: footprint (none) -> Resistors_THT:R_Axial_DIN0207_L6.3mm_D2.5mm_P10.16mm_Horizontal
- RV1: footprint Potentiometers:Potentiometer_Alps-RK16-single -> Potentiometers:Potentiometer_Alps_RK09K_Horizontal
- U1: footprint TO_SOT_Packages_THT:TO-220_Neutral123_PadsOnly -> TO_SOT_Packages_THT:TO-92_Inline_Narrow_Oval
- U2, U3, U7: footprint Housings_DIP:DIP-8_W7.62mm -> Housings_DIP:DIP-8_W7.62mm_LongPads
- U4: footprint TO_SOT_Packages_THT:TO-92_Inline_Wide -> TO_SOT_Packages_THT:TO-92_Inline_Narrow_Oval
- U5: footprint TO-220 -> TO_SOT_Packages_THT:TO-92_Inline_Narrow_Oval
- U6: footprint Socket_Strips:Socket_Strip_Straight_1x38 -> Pin_Headers:Pin_Header_Straight_2x25_Pitch2.54mm
- U8: footprint Socket_Strips:Socket_Strip_Straight_1x04 -> Pin_Headers:Pin_Header_Straight_1x04_Pitch2.54mm
- U9: footprint kaini:QFP48 Adapter -> Housings_QFP:LQFP-48_7x7mm_Pitch0.5mm
- Y1: footprint Crystals:Crystal_Round_d3.0mm_Vertical -> Crystals:Crystal_AT310_d3.0mm_l10.0mm_Vertical
Connections:
- net DCL: now also U9.29 (PIO0_14); no longer U9.23 (PIO0_8)
- net DD0: now also U9.22 (PIO0_7); no longer U9.15 (PIO0_0)
- net DD1: now also U9.21 (PIO0_6); no longer U9.16 (PIO0_1)
- net DD2: now also U9.20 (PIO0_5); no longer U9.17 (PIO0_2)
- net DD3: now also U9.19 (PIO0_4); no longer U9.18 (PIO0_3)
- net DD4: now also U9.18 (PIO0_3); no longer U9.19 (PIO0_4)
- net DD5: now also U9.17 (PIO0_2); no longer U9.20 (PIO0_5)
- net DD6: now also U9.16 (PIO0_1); no longer U9.21 (PIO0_6)
- net DD7: now also U9.15 (PIO0_0); no longer U9.22 (PIO0_7)
- net DGMODE: now also U9.32 (PIO0_17); no longer U9.29 (PIO0_14)
- net DLE: now also U9.25 (PIO0_10); no longer U9.24 (PIO0_9)
- net DOE: now also U9.24 (PIO0_9); no longer U9.25 (PIO0_10)
- net DON: now also U9.14 (PIO0_29*); no longer U9.13 (PIO0_28*)
- net DSPH: now also U9.23 (PIO0_8); no longer U9.32 (PIO0_17)
- net TON: now also U9.12 (PIO0_27*); no longer U9.14 (PIO0_29*)
- net at R12.2: now also Q3.3 (S); no longer Q3.2 (D)
- net at C4.1, Q1.1 (G), R1.1: now also Q3.2 (D); no longer Q3.3 (S)
- net at R13.2: now also Q4.3 (S); no longer Q4.2 (D)
- net at C5.1, Q2.1 (G), R3.1: now also Q4.2 (D); no longer Q4.3 (S)
