File: kicad/eink.sch (KiCad schematic (older format))
At the start: 6 parts, among them U7 LM358, U8 ED060SC4V2

Commit message: Finish schematic
Parts:
- removed U7: LM358, symbol LM358
- added U3: TS321ILT, symbol TS881
- renumbered C18 to C10, C17 to C9, R12 to R4, RV2 to RV1, U8 to U4
Connections:
- wire segments 53 -> 57
Changed lines of the file:
@@
 $Descr A4 11693 8268
 encoding utf-8
-Sheet 5 5
-Title ""
-Date ""
-Rev ""
+Sheet 3 5
+Title "E-Ink Clock"
+Date "2017-03-29"
+Rev "1.0"
 Comp ""
 Comment1 ""
@@
 $EndDescr
 $Comp
-L ED060SC4V2 U8
+L ED060SC4V2 U4
 U 1 1 58E0CC09
 P 2900 5100
-F 0 "U8" H 3600 4250 60  0000 R CNN
+F 0 "U4" H 3600 4250 60  0000 R CNN
 F 1 "ED060SC4V2" H 2900 5100 60  0000 C CNN
 F 2 "" H 3200 5250 60  0001 C CNN
@@
 $EndComp
 $Comp
-L LM358 U7
-U 2 1 58E0CC24
-P 2300 2250
-F 0 "U7" H 2300 2450 50  0000 L CNN
-F 1 "LM358" H 2300 2050 50  0000 L CNN
-F 2 "" H 2300 2250 50  0001 C CNN
-F 3 "" H 2300 2250 50  0000 C CNN
-	2    2300 2250
-	1    0    0    1
-$EndComp
-$Comp
-L C C17
+L C C9
 U 1 1 58E0CC2B
 P 3050 2500
-F 0 "C17" H 3075 2600 50  0000 L CNN
+F 0 "C9" H 3075 2600 50  0000 L CNN
 F 1 "100n" H 3075 2400 50  0000 L CNN
 F 2 "" H 3088 2350 50  0001 C CNN
@@
 $EndComp
 $Comp
-L GND #PWR06
+L GND #PWR11
 U 1 1 58E0CC32
 P 3300 2600
-F 0 "#PWR06" H 3300 2350 50  0001 C CNN
+F 0 "#PWR11" H 3300 2350 50  0001 C CNN
 F 1 "GND" H 3300 2450 50  0000 C CNN
 F 2 "" H 3300 2600 50  0000 C CNN
@@
 $EndComp
 $Comp
-L R R12
+L R R4
 U 1 1 58E0CC3A
 P 1650 1950
-F 0 "R12" V 1730 1950 50  0000 C CNN
+F 0 "R4" V 1730 1950 50  0000 C CNN
 F 1 "47k" V 1650 1950 50  0000 C CNN
 F 2 "" V 1580 1950 50  0001 C CNN
@@
 $EndComp
 $Comp
-L POT RV2
+L POT RV1
 U 1 1 58E0CC41
 P 1650 2350
-F 0 "RV2" V 1475 2350 50  0000 C CNN
+F 0 "RV1" V 1475 2350 50  0000 C CNN
 F 1 "10k" V 1550 2350 50  0000 C CNN
 F 2 "" H 1650 2350 50  0001 C CNN
@@
 $EndComp
 $Comp
-L GND #PWR07
+L GND #PWR7
 U 1 1 58E0CC48
 P 1650 2600
-F 0 "#PWR07" H 1650 2350 50  0001 C CNN
+F 0 "#PWR7" H 1650 2350 50  0001 C CNN
 F 1 "GND" H 1650 2450 50  0000 C CNN
 F 2 "" H 1650 2600 50  0000 C CNN
@@
 	2200 2550 2200 2850
 Wire Wire Line
-	2200 1600 2200 1950
+	2200 1600 2200 1700
+Wire Wire Line
+	2200 1700 2200 1950
 Wire Wire Line
 	2800 1900 1900 1900
@@
 Connection ~ 2800 2500
 $Comp
-L GND #PWR08
+L GND #PWR10
 U 1 1 58E0CC71
 P 2900 6500
-F 0 "#PWR08" H 2900 6250 50  0001 C CNN
+F 0 "#PWR10" H 2900 6250 50  0001 C CNN
 F 1 "GND" H 2900 6350 50  0000 C CNN
 F 2 "" H 2900 6500 50  0000 C CNN
@@
 	2000 4900 2100 4900
 $Comp
-L GND #PWR09
+L GND #PWR8
 U 1 1 58E0CC80
 P 1650 5000
-F 0 "#PWR09" H 1650 4750 50  0001 C CNN
+F 0 "#PWR8" H 1650 4750 50  0001 C CNN
 F 1 "GND" H 1650 4850 50  0000 C CNN
 F 2 "" H 1650 5000 50  0000 C CNN
@@
 	2000 5200 2100 5200
 $Comp
-L GND #PWR010
+L GND #PWR9
 U 1 1 58E0CC89
 P 2700 4100
-F 0 "#PWR010" H 2700 3850 50  0001 C CNN
+F 0 "#PWR9" H 2700 3850 50  0001 C CNN
 F 1 "GND" H 2700 3950 50  0000 C CNN
 F 2 "" H 2700 4100 50  0000 C CNN
@@
 	2900 6500 2900 6000
 Wire Wire Line
-	2800 1900 2800 4200
+	2800 1900 2800 2250
+Wire Wire Line
+	2800 2250 2800 2500
+Wire Wire Line
+	2800 2500 2800 4200
 Wire Wire Line
 	2900 4100 2900 4200
 Wire Wire Line
-	3000 3550 3000 4200
+	3000 3550 3000 3700
+Wire Wire Line
+	3000 3700 3000 4200
 Wire Wire Line
 	3100 4100 3100 4200
@@
 	3800 5800 3700 5800
 $Comp
-L GND #PWR011
+L GND #PWR13
 U 1 1 58E0CCA1
 P 4150 4800
-F 0 "#PWR011" H 4150 4550 50  0001 C CNN
+F 0 "#PWR13" H 4150 4550 50  0001 C CNN
 F 1 "GND" H 4150 4650 50  0000 C CNN
 F 2 "" H 4150 4800 50  0000 C CNN
@@
 $EndComp
 $Comp
-L C C18
+L C C10
 U 1 1 58E0CCA8
 P 3250 3700
-F 0 "C18" H 3275 3800 50  0000 L CNN
+F 0 "C10" H 3275 3800 50  0000 L CNN
 F 1 "100n" H 3275 3600 50  0000 L CNN
 F 2 "" H 3288 3550 50  0001 C CNN
@@
 Connection ~ 3000 3700
 $Comp
-L GND #PWR012
+L GND #PWR12
 U 1 1 58E0F8B1
 P 3500 3800
-F 0 "#PWR012" H 3500 3550 50  0001 C CNN
+F 0 "#PWR12" H 3500 3550 50  0001 C CNN
 F 1 "GND" H 3500 3650 50  0000 C CNN
 F 2 "" H 3500 3800 50  0000 C CNN
@@
 Text HLabel 3800 5800 2    60   Input ~ 0
 DD7
+$Comp
+L TS881 U3
+U 1 1 58DE29E1
+P 2300 2250
+F 0 "U3" H 2300 2500 50  0000 L CNN
+F 1 "TS321ILT" H 2300 2400 50  0000 L CNN
+F 2 "" H 2300 2250 50  0001 C CNN
+F 3 "" H 2300 2250 50  0001 C CNN
+	1    2300 2250
+	1    0    0    1
+$EndComp
 $EndSCHEMATC

Commit message: Set most footprints
Parts:
- C10, C9: footprint (none) -> Capacitors_SMD:C_0805_HandSoldering
- R4: footprint (none) -> Resistors_SMD:R_0805_HandSoldering
- U3: footprint (none) -> TO_SOT_Packages_SMD:SOT-23-5_HandSoldering
- U4: footprint (none) -> einkclock:Hirose_FH26-39S-0.3SHW
Changed lines of the file:
@@
 F 0 "U4" H 3600 4250 60  0000 R CNN
 F 1 "ED060SC4V2" H 2900 5100 60  0000 C CNN
-F 2 "" H 3200 5250 60  0001 C CNN
+F 2 "einkclock:Hirose_FH26-39S-0.3SHW" H 3200 5250 60  0001 C CNN
 F 3 "" H 3200 5250 60  0001 C CNN
 	1    2900 5100
@@
 F 0 "C9" H 3075 2600 50  0000 L CNN
 F 1 "100n" H 3075 2400 50  0000 L CNN
-F 2 "" H 3088 2350 50  0001 C CNN
+F 2 "Capacitors_SMD:C_0805_HandSoldering" H 3088 2350 50  0001 C CNN
 F 3 "" H 3050 2500 50  0000 C CNN
 	1    3050 2500
@@
 $EndComp
 $Comp
-L GND #PWR11
+L GND #PWR07
 U 1 1 58E0CC32
 P 3300 2600
-F 0 "#PWR11" H 3300 2350 50  0001 C CNN
+F 0 "#PWR07" H 3300 2350 50  0001 C CNN
 F 1 "GND" H 3300 2450 50  0000 C CNN
 F 2 "" H 3300 2600 50  0000 C CNN
@@
 F 0 "R4" V 1730 1950 50  0000 C CNN
 F 1 "47k" V 1650 1950 50  0000 C CNN
-F 2 "" V 1580 1950 50  0001 C CNN
+F 2 "Resistors_SMD:R_0805_HandSoldering" V 1580 1950 50  0001 C CNN
 F 3 "" H 1650 1950 50  0000 C CNN
 	1    1650 1950
@@
 $EndComp
 $Comp
-L GND #PWR7
+L GND #PWR08
 U 1 1 58E0CC48
 P 1650 2600
-F 0 "#PWR7" H 1650 2350 50  0001 C CNN
+F 0 "#PWR08" H 1650 2350 50  0001 C CNN
 F 1 "GND" H 1650 2450 50  0000 C CNN
 F 2 "" H 1650 2600 50  0000 C CNN
@@
 	2200 2550 2200 2850
 Wire Wire Line
-	2200 1600 2200 1700
-Wire Wire Line
-	2200 1700 2200 1950
+	2200 1600 2200 1950
 Wire Wire Line
 	2800 1900 1900 1900
@@
 Connection ~ 2800 2500
 $Comp
-L GND #PWR10
+L GND #PWR09
 U 1 1 58E0CC71
 P 2900 6500
-F 0 "#PWR10" H 2900 6250 50  0001 C CNN
+F 0 "#PWR09" H 2900 6250 50  0001 C CNN
 F 1 "GND" H 2900 6350 50  0000 C CNN
 F 2 "" H 2900 6500 50  0000 C CNN
@@
 	2000 4900 2100 4900
 $Comp
-L GND #PWR8
+L GND #PWR010
 U 1 1 58E0CC80
 P 1650 5000
-F 0 "#PWR8" H 1650 4750 50  0001 C CNN
+F 0 "#PWR010" H 1650 4750 50  0001 C CNN
 F 1 "GND" H 1650 4850 50  0000 C CNN
 F 2 "" H 1650 5000 50  0000 C CNN
@@
 	2000 5200 2100 5200
 $Comp
-L GND #PWR9
+L GND #PWR011
 U 1 1 58E0CC89
 P 2700 4100
-F 0 "#PWR9" H 2700 3850 50  0001 C CNN
+F 0 "#PWR011" H 2700 3850 50  0001 C CNN
 F 1 "GND" H 2700 3950 50  0000 C CNN
 F 2 "" H 2700 4100 50  0000 C CNN
@@
 	2900 6500 2900 6000
 Wire Wire Line
-	2800 1900 2800 2250
-Wire Wire Line
-	2800 2250 2800 2500
-Wire Wire Line
-	2800 2500 2800 4200
+	2800 1900 2800 4200
 Wire Wire Line
 	2900 4100 2900 4200
 Wire Wire Line
-	3000 3550 3000 3700
-Wire Wire Line
-	3000 3700 3000 4200
+	3000 3550 3000 4200
 Wire Wire Line
 	3100 4100 3100 4200
@@
 	3800 5800 3700 5800
 $Comp
-L GND #PWR13
+L GND #PWR012
 U 1 1 58E0CCA1
 P 4150 4800
-F 0 "#PWR13" H 4150 4550 50  0001 C CNN
+F 0 "#PWR012" H 4150 4550 50  0001 C CNN
 F 1 "GND" H 4150 4650 50  0000 C CNN
 F 2 "" H 4150 4800 50  0000 C CNN
@@
 F 0 "C10" H 3275 3800 50  0000 L CNN
 F 1 "100n" H 3275 3600 50  0000 L CNN
-F 2 "" H 3288 3550 50  0001 C CNN
+F 2 "Capacitors_SMD:C_0805_HandSoldering" H 3288 3550 50  0001 C CNN
 F 3 "" H 3250 3700 50  0000 C CNN
 	1    3250 3700
@@
 Connection ~ 3000 3700
 $Comp
-L GND #PWR12
+L GND #PWR013
 U 1 1 58E0F8B1
 P 3500 3800
-F 0 "#PWR12" H 3500 3550 50  0001 C CNN
+F 0 "#PWR013" H 3500 3550 50  0001 C CNN
 F 1 "GND" H 3500 3650 50  0000 C CNN
 F 2 "" H 3500 3800 50  0000 C CNN
@@
 F 0 "U3" H 2300 2500 50  0000 L CNN
 F 1 "TS321ILT" H 2300 2400 50  0000 L CNN
-F 2 "" H 2300 2250 50  0001 C CNN
+F 2 "TO_SOT_Packages_SMD:SOT-23-5_HandSoldering" H 2300 2250 50  0001 C CNN
 F 3 "" H 2300 2250 50  0001 C CNN
 	1    2300 2250

Commit message: Finish footprints
Parts:
- RV1: footprint (none) -> Potentiometers:Potentiometer_Trimmer_Vishay_TS53YL
Changed lines of the file:
@@
 F 0 "RV1" V 1475 2350 50  0000 C CNN
 F 1 "10k" V 1550 2350 50  0000 C CNN
-F 2 "" H 1650 2350 50  0001 C CNN
+F 2 "Potentiometers:Potentiometer_Trimmer_Vishay_TS53YL" H 1650 2350 50  0001 C CNN
 F 3 "" H 1650 2350 50  0000 C CNN
 	1    1650 2350

Commit message: First routing
Parts:
- C10, C9: footprint Capacitors_SMD:C_0805_HandSoldering -> Resistors_SMD:R_0805_HandSoldering
Changed lines of the file:
@@
 F 0 "C9" H 3075 2600 50  0000 L CNN
 F 1 "100n" H 3075 2400 50  0000 L CNN
-F 2 "Capacitors_SMD:C_0805_HandSoldering" H 3088 2350 50  0001 C CNN
+F 2 "Resistors_SMD:R_0805_HandSoldering" H 3088 2350 50  0001 C CNN
 F 3 "" H 3050 2500 50  0000 C CNN
 	1    3050 2500
@@
 F 0 "C10" H 3275 3800 50  0000 L CNN
 F 1 "100n" H 3275 3600 50  0000 L CNN
-F 2 "Capacitors_SMD:C_0805_HandSoldering" H 3288 3550 50  0001 C CNN
+F 2 "Resistors_SMD:R_0805_HandSoldering" H 3288 3550 50  0001 C CNN
 F 3 "" H 3250 3700 50  0000 C CNN
 	1    3250 3700

Commit message: Add BOM
Parts:
- C10, C9: Manf# (none) -> 885012207098
- R4: Manf# (none) -> ERJ-6GEYJ473V
- RV1: Manf# (none) -> TS53YL103MR10
- U3: Manf# (none) -> TS321ILT
- U4: Manf# (none) -> FH26W-39S-0.3SHW(98)
Changed lines of the file:
@@
 F 2 "einkclock:Hirose_FH26-39S-0.3SHW" H 3200 5250 60  0001 C CNN
 F 3 "" H 3200 5250 60  0001 C CNN
+F 4 "FH26W-39S-0.3SHW(98)" H 2900 5100 60  0001 C CNN "Manf#"
 	1    2900 5100
 	1    0    0    -1
@@
 F 2 "Resistors_SMD:R_0805_HandSoldering" H 3088 2350 50  0001 C CNN
 F 3 "" H 3050 2500 50  0000 C CNN
+F 4 "885012207098" H 3050 2500 60  0001 C CNN "Manf#"
 	1    3050 2500
 	0    -1   1    0
@@
 F 2 "Resistors_SMD:R_0805_HandSoldering" V 1580 1950 50  0001 C CNN
 F 3 "" H 1650 1950 50  0000 C CNN
+F 4 "ERJ-6GEYJ473V" V 1650 1950 60  0001 C CNN "Manf#"
 	1    1650 1950
 	1    0    0    1
@@
 F 2 "Potentiometers:Potentiometer_Trimmer_Vishay_TS53YL" H 1650 2350 50  0001 C CNN
 F 3 "" H 1650 2350 50  0000 C CNN
+F 4 "TS53YL103MR10" V 1650 2350 60  0001 C CNN "Manf#"
 	1    1650 2350
 	1    0    0    1
@@
 F 2 "Resistors_SMD:R_0805_HandSoldering" H 3288 3550 50  0001 C CNN
 F 3 "" H 3250 3700 50  0000 C CNN
+F 4 "885012207098" H 3250 3700 60  0001 C CNN "Manf#"
 	1    3250 3700
 	0    -1   -1   0
@@
 F 2 "TO_SOT_Packages_SMD:SOT-23-5_HandSoldering" H 2300 2250 50  0001 C CNN
 F 3 "" H 2300 2250 50  0001 C CNN
+F 4 "TS321ILT" H 2300 2250 60  0001 C CNN "Manf#"
 	1    2300 2250
 	1    0    0    1
