File: kicad/cpu.sch (KiCad schematic (older format))
At the start: 15 parts, among them P1 SWD, U1 23LC512, U2 LPC1227FBD48/301, Y1 32.768k 12.5p

Commit message: First routing
Parts:
- C1, C2, C3, C4, C5, C6, C7, C8: footprint Capacitors_SMD:C_0805_HandSoldering -> Resistors_SMD:R_0805_HandSoldering
Connections:
- net DCKV: now also U2.25 (PIO0_10); no longer U2.5 (PIO0_20)
- net DCL: now also U2.5 (PIO0_20); no longer U2.23 (PIO0_8)
- net DGMODE: now also U2.23 (PIO0_8); no longer U2.7 (PIO0_22)
- net DLE: now also U2.6 (PIO0_21); no longer U2.24 (PIO0_9)
- net DOE: now also U2.7 (PIO0_22); no longer U2.25 (PIO0_10)
- net DON: now also U2.14 (PIO0_29*); no longer U2.13 (PIO0_28*)
- net DSPH: now also U2.8 (PIO0_23); no longer U2.6 (PIO0_21)
- net DSPV: now also U2.24 (PIO0_9); no longer U2.8 (PIO0_23)
- net TON: now also U2.13 (PIO0_28*); no longer U2.14 (PIO0_29*)
- net at C8.1, U2.45 (RTCXOUT): now also Y1.1; no longer Y1.2
- net at C5.1, U2.46 (RTCXIN): now also Y1.2; no longer Y1.1
Changed lines of the file:
@@
 F 0 "C6" H 6725 3850 50  0000 L CNN
 F 1 "100n" H 6725 3650 50  0000 L CNN
-F 2 "Capacitors_SMD:C_0805_HandSoldering" H 6738 3600 50  0001 C CNN
+F 2 "Resistors_SMD:R_0805_HandSoldering" H 6738 3600 50  0001 C CNN
 F 3 "" H 6700 3750 50  0000 C CNN
 	1    6700 3750
@@
 F 0 "C7" H 6975 3850 50  0000 L CNN
 F 1 "100n" H 6975 3650 50  0000 L CNN
-F 2 "Capacitors_SMD:C_0805_HandSoldering" H 6988 3600 50  0001 C CNN
+F 2 "Resistors_SMD:R_0805_HandSoldering" H 6988 3600 50  0001 C CNN
 F 3 "" H 6950 3750 50  0000 C CNN
 	1    6950 3750
@@
 F 3 "" H 6750 4300 50  0000 C CNN
 	1    6750 4300
-	1    0    0    -1
+	-1   0    0    -1
 $EndComp
 $Comp
@@
 F 0 "C5" H 6475 4800 50  0000 L CNN
 F 1 "22p" H 6475 4600 50  0000 L CNN
-F 2 "Capacitors_SMD:C_0805_HandSoldering" H 6488 4550 50  0001 C CNN
+F 2 "Resistors_SMD:R_0805_HandSoldering" H 6488 4550 50  0001 C CNN
 F 3 "" H 6450 4700 50  0000 C CNN
 	1    6450 4700
@@
 F 0 "C8" H 7075 4800 50  0000 L CNN
 F 1 "22p" H 7075 4600 50  0000 L CNN
-F 2 "Capacitors_SMD:C_0805_HandSoldering" H 7088 4550 50  0001 C CNN
+F 2 "Resistors_SMD:R_0805_HandSoldering" H 7088 4550 50  0001 C CNN
 F 3 "" H 7050 4700 50  0000 C CNN
 	1    7050 4700
@@
 F 0 "C1" H 2275 4650 50  0000 L CNN
 F 1 "100n" H 2275 4450 50  0000 L CNN
-F 2 "Capacitors_SMD:C_0805_HandSoldering" H 2288 4400 50  0001 C CNN
+F 2 "Resistors_SMD:R_0805_HandSoldering" H 2288 4400 50  0001 C CNN
 F 3 "" H 2250 4550 50  0000 C CNN
 	1    2250 4550
@@
 F 0 "C3" H 3575 3250 50  0000 L CNN
 F 1 "100n" H 3575 3050 50  0000 L CNN
-F 2 "Capacitors_SMD:C_0805_HandSoldering" H 3588 3000 50  0001 C CNN
+F 2 "Resistors_SMD:R_0805_HandSoldering" H 3588 3000 50  0001 C CNN
 F 3 "" H 3550 3150 50  0000 C CNN
 	1    3550 3150
@@
 F 0 "C4" H 6475 3850 50  0000 L CNN
 F 1 "4.7µ" H 6475 3650 50  0000 L CNN
-F 2 "Capacitors_SMD:C_0805_HandSoldering" H 6488 3600 50  0001 C CNN
+F 2 "Resistors_SMD:R_0805_HandSoldering" H 6488 3600 50  0001 C CNN
 F 3 "" H 6450 3750 50  0000 C CNN
 	1    6450 3750
@@
 Text HLabel 4700 2200 0    60   Input ~ 0
 DD7
-Text HLabel 4700 2400 0    60   Input ~ 0
+Text HLabel 4700 3700 0    60   Input ~ 0
 DCL
-Text HLabel 4700 2500 0    60   Input ~ 0
+Text HLabel 4700 3800 0    60   Input ~ 0
 DLE
-Text HLabel 4700 2600 0    60   Input ~ 0
+Text HLabel 4700 3900 0    60   Input ~ 0
 DOE
 Text HLabel 4700 2700 0    60   Input ~ 0
@@
 Text HLabel 7150 4000 2    60   Input ~ 0
 +3.3V
-Text HLabel 4700 3900 0    60   Input ~ 0
+Text HLabel 4700 2400 0    60   Input ~ 0
 DGMODE
+Text HLabel 4700 2500 0    60   Input ~ 0
+DSPV
+Text HLabel 4700 2600 0    60   Input ~ 0
+DCKV
 Text HLabel 4700 4000 0    60   Input ~ 0
-DSPV
-Text HLabel 4700 3700 0    60   Input ~ 0
-DCKV
-Text HLabel 4700 3800 0    60   Input ~ 0
 DSPH
 Text HLabel 4700 3500 0    60   Input ~ 0
@@
 Text HLabel 4700 3600 0    60   Input ~ 0
 ONNEG
+Text HLabel 4700 4700 0    60   Input ~ 0
+DON
 Text HLabel 4700 4600 0    60   Input ~ 0
-DON
-Text HLabel 4700 4700 0    60   Input ~ 0
 TON
 Wire Wire Line
@@
 F 0 "C2" H 3275 1400 50  0000 L CNN
 F 1 "100n" H 3275 1200 50  0000 L CNN
-F 2 "Capacitors_SMD:C_0805_HandSoldering" H 3288 1150 50  0001 C CNN
+F 2 "Resistors_SMD:R_0805_HandSoldering" H 3288 1150 50  0001 C CNN
 F 3 "" H 3250 1300 50  0001 C CNN
 	1    3250 1300

Commit message: Add BOM
Parts:
- C1, C2, C3, C6, C7: Manf# (none) -> 885012207098
- C4: Manf# (none) -> GRM21BR61E475MA12L
- C5, C8: Manf# (none) -> 885012007053
- R1, R2, R3: Manf# (none) -> AS08J1002ET
- U1: Manf# (none) -> 23LC512-I/SN
- U2: Manf# (none) -> LPC1227FBD48/301,1
- Y1: Manf# (none) -> AB26TRQ-32.768kHz-T
Changed lines of the file:
@@
 F 2 "Housings_QFP:LQFP-48_7x7mm_Pitch0.5mm" H 5300 4850 60  0001 C CNN
 F 3 "" H 5300 4850 60  0001 C CNN
+F 4 "LPC1227FBD48/301,1" H 5500 3600 60  0001 C CNN "Manf#"
 	1    5500 3600
 	1    0    0    -1
@@
 F 2 "Resistors_SMD:R_0805_HandSoldering" H 6738 3600 50  0001 C CNN
 F 3 "" H 6700 3750 50  0000 C CNN
+F 4 "885012207098" H 6700 3750 60  0001 C CNN "Manf#"
 	1    6700 3750
 	1    0    0    -1
@@
 F 2 "Resistors_SMD:R_0805_HandSoldering" H 6988 3600 50  0001 C CNN
 F 3 "" H 6950 3750 50  0000 C CNN
+F 4 "885012207098" H 6950 3750 60  0001 C CNN "Manf#"
 	1    6950 3750
 	1    0    0    -1
@@
 F 2 "einkclock:Crystal_Lying_1" H 6750 4300 50  0001 C CNN
 F 3 "" H 6750 4300 50  0000 C CNN
+F 4 "AB26TRQ-32.768kHz-T" H 6750 4300 60  0001 C CNN "Manf#"
 	1    6750 4300
 	-1   0    0    -1
@@
 F 2 "Resistors_SMD:R_0805_HandSoldering" H 6488 4550 50  0001 C CNN
 F 3 "" H 6450 4700 50  0000 C CNN
+F 4 "885012007053" H 6450 4700 60  0001 C CNN "Manf#"
 	1    6450 4700
 	1    0    0    -1
@@
 F 2 "Resistors_SMD:R_0805_HandSoldering" H 7088 4550 50  0001 C CNN
 F 3 "" H 7050 4700 50  0000 C CNN
+F 4 "885012007053" H 7050 4700 60  0001 C CNN "Manf#"
 	1    7050 4700
 	1    0    0    -1
@@
 F 2 "Resistors_SMD:R_0805_HandSoldering" V 3480 2650 50  0001 C CNN
 F 3 "" H 3550 2650 50  0000 C CNN
+F 4 "AS08J1002ET" V 3550 2650 60  0001 C CNN "Manf#"
 	1    3550 2650
 	-1   0    0    1
@@
 F 2 "Resistors_SMD:R_0805_HandSoldering" H 2288 4400 50  0001 C CNN
 F 3 "" H 2250 4550 50  0000 C CNN
+F 4 "885012207098" H 2250 4550 60  0001 C CNN "Manf#"
 	1    2250 4550
 	-1   0    0    1
@@
 F 2 "Resistors_SMD:R_0805_HandSoldering" H 3588 3000 50  0001 C CNN
 F 3 "" H 3550 3150 50  0000 C CNN
+F 4 "885012207098" H 3550 3150 60  0001 C CNN "Manf#"
 	1    3550 3150
 	-1   0    0    1
@@
 F 2 "Resistors_SMD:R_0805_HandSoldering" V 3730 4800 50  0001 C CNN
 F 3 "" H 3800 4800 50  0000 C CNN
+F 4 "AS08J1002ET" V 3800 4800 60  0001 C CNN "Manf#"
 	1    3800 4800
 	-1   0    0    1
@@
 F 2 "Resistors_SMD:R_0805_HandSoldering" V 3930 4800 50  0001 C CNN
 F 3 "" H 4000 4800 50  0000 C CNN
+F 4 "AS08J1002ET" V 4000 4800 60  0001 C CNN "Manf#"
 	1    4000 4800
 	-1   0    0    1
@@
 F 2 "Resistors_SMD:R_0805_HandSoldering" H 6488 3600 50  0001 C CNN
 F 3 "" H 6450 3750 50  0000 C CNN
+F 4 "GRM21BR61E475MA12L" H 6450 3750 60  0001 C CNN "Manf#"
 	1    6450 3750
 	1    0    0    -1
@@
 F 2 "Resistors_SMD:R_0805_HandSoldering" H 3288 1150 50  0001 C CNN
 F 3 "" H 3250 1300 50  0001 C CNN
+F 4 "885012207098" H 3250 1300 60  0001 C CNN "Manf#"
 	1    3250 1300
 	1    0    0    -1
@@
 F 2 "Housings_SOIC:SOIC-8_3.9x4.9mm_Pitch1.27mm" H 2150 1200 60  0001 C CNN
 F 3 "" H 2150 1200 60  0001 C CNN
+F 4 "23LC512-I/SN" H 2150 1200 60  0001 C CNN "Manf#"
 	1    2150 1200
 	1    0    0    -1

Commit message: Finish BOM and fix PCB according to the parts
Parts:
- P1: Manf# (none) -> 61201021621
Changed lines of the file:
@@
 F 2 "Connectors:IDC_Header_Straight_10pins" H 3050 3300 50  0001 C CNN
 F 3 "" H 3050 3300 50  0000 C CNN
+F 4 "61201021621" H 3050 4500 60  0001 C CNN "Manf#"
 	1    3050 4500
 	1    0    0    -1
